File: kicad/PedalComposer.kicad_pcb (KiCad board)
At the start: 2 copper layers, 81 parts, among them J1 In, J10 Fx5In, J11 Fx5Out, J12 Fx6In, J13 Fx6Out, J14 Out, J15 Jack-DC, J2 Fx1In, J3 Fx1Out, J4 Fx2In, J5 Fx2Out, J6 Fx3In, J7 Fx3Out, J8 Fx4In, J9 Fx4Out, SW1 Fx1, SW11 Edit, SW12 All, SW2 Fx2, SW3 Fx3, SW4 Fx4, SW5 Fx5, SW6 Fx6, U1 LM317L_TO92, U10 CD4053B, U2 LM317L_TO92, U20 CD4053B, U30 CD4053B, U40 CD4053B, U5 ATmega8535-16P, Y1 12MHz

Commit message: WIP layout
Parts:
- removed J11: Fx5Out, BDMLibrary:Mono Female Socket Connector
- removed J12: Fx6In, BDMLibrary:Mono Female Socket Connector
- removed J13: Fx6Out, BDMLibrary:Mono Female Socket Connector
- removed R25, R27, R28, R29, R31: 1M, Resistor_THT:R_Axial_DIN0207_L6.3mm_D2.5mm_P7.62mm_Horizontal
- removed SW12: All, BDMLibrary:SW_Toggle_Blue_wSlots
- removed SW5: Fx5, BDMLibrary:SW_Toggle_Blue_wSlots
- removed SW6: Fx6, BDMLibrary:SW_Toggle_Blue_wSlots
- removed U40: CD4053B, Package_DIP:DIP-16_W7.62mm_Socket
- added D10: Ctrl2, LED_THT:LED_D3.0mm, F.Cu at (108.6, 73.5)
- added D11: Ctrl3, LED_THT:LED_D3.0mm, F.Cu at (48.1, 73.5)
- added D9: Ctrl1, LED_THT:LED_D3.0mm, F.Cu at (169.0, 73.5)
- added M1: 7-SEGMENT-1DIGIT-1INCH-BLUE, Display_7Segment:7SegmentLED_LTS6760_LTS6780, F.Cu at (211.3, 68.1)
- added R32: 470, Resistor_SMD:R_0603_1608Metric, F.Cu at (226.3, 51.8)
- added R33: 470, Resistor_SMD:R_0603_1608Metric, F.Cu at (234.2, 55.9)
- added R34: 470, Resistor_SMD:R_0603_1608Metric, F.Cu at (212.3, 79.8)
- added R35: 470, Resistor_SMD:R_0603_1608Metric, F.Cu at (205.2, 80.0)
- added R36: 470, Resistor_SMD:R_0603_1608Metric, F.Cu at (205.2, 69.8)
- added R37: 470, Resistor_SMD:R_0603_1608Metric, F.Cu at (213.1, 47.4)
- added R38: 470, Resistor_SMD:R_0603_1608Metric, F.Cu at (199.9, 58.4)
- added R39: 470, Resistor_SMD:R_0603_1608Metric, F.Cu at (216.9, 72.1)
- added U3: 4543, Package_SO:SOIC-16_4.55x10.3mm_P1.27mm, F.Cu at (193.0, 73.2)
- C1: value 100pF -> 100nF; footprint Capacitor_THT:C_Disc_D5.0mm_W2.5mm_P5.00mm -> Capacitor_SMD:C_0603_1608Metric
- C10, C11, C9: footprint Capacitor_THT:C_Rect_L7.2mm_W3.0mm_P5.00mm_FKS2_FKP2_MKS2_MKP2 -> Capacitor_SMD:C_0603_1608Metric
- C12, C7: footprint Capacitor_THT:C_Rect_L7.2mm_W3.0mm_P5.00mm_FKS2_FKP2_MKS2_MKP2 -> Capacitor_SMD:C_0603_1608Metric; moved to B.Cu
- C13, C8: footprint Capacitor_THT:C_Rect_L7.2mm_W3.0mm_P5.00mm_FKS2_FKP2_MKS2_MKP2 -> Capacitor_SMD:C_Elec_4x5.4
- C2, C4: footprint Capacitor_THT:C_Radial_D6.3mm_H11.0mm_P2.50mm -> Capacitor_SMD:C_Elec_4x5.4
- C3: value 100pF -> 10nF; footprint Capacitor_THT:C_Disc_D5.0mm_W2.5mm_P5.00mm -> Capacitor_SMD:C_0603_1608Metric
- C5, C6: footprint Capacitor_THT:C_Disc_D5.0mm_W2.5mm_P5.00mm -> Capacitor_SMD:C_0603_1608Metric
- D1: value LED -> Fx1
- D2: value LED -> Fx2
- D3: value LED -> Fx3
- D4: value LED -> Fx4
- D5, D6: footprint LED_THT:LED_D3.0mm -> LED_SMD:LED_0603_1608Metric
- J1, J14: footprint BDMLibrary:Mono Female Socket Connector -> BDMLibrary:Mono Female Socket Connector TS
- J10: value Fx5In -> AVR-ISP-6; footprint BDMLibrary:Mono Female Socket Connector -> Connector_PinHeader_2.54mm:PinHeader_2x03_P2.54mm_Vertical
- J2: value Fx1In -> Send1; footprint BDMLibrary:Mono Female Socket Connector -> BDMLibrary:Mono Female Socket Connector TS
- J3: value Fx1Out -> Return1; footprint BDMLibrary:Mono Female Socket Connector -> BDMLibrary:Mono Female Socket Connector TS
- J4: value Fx2In -> Send2; footprint BDMLibrary:Mono Female Socket Connector -> BDMLibrary:Mono Female Socket Connector TS
- J5: value Fx2Out -> Return2; footprint BDMLibrary:Mono Female Socket Connector -> BDMLibrary:Mono Female Socket Connector TS
- J6: value Fx3In -> Send3; footprint BDMLibrary:Mono Female Socket Connector -> BDMLibrary:Mono Female Socket Connector TS
- J7: value Fx3Out -> Return3; footprint BDMLibrary:Mono Female Socket Connector -> BDMLibrary:Mono Female Socket Connector TS
- J8: value Fx4In -> Send4; footprint BDMLibrary:Mono Female Socket Connector -> BDMLibrary:Mono Female Socket Connector TS
- J9: value Fx4Out -> Return4; footprint BDMLibrary:Mono Female Socket Connector -> BDMLibrary:Mono Female Socket Connector TS
- R1, R10, R11, R12, R13, R14, R16, R17, R18, R19, R2, R20, R21, R22, R26, R3, R30, R4, R5, R6, R7, R8, R9: footprint Resistor_THT:R_Axial_DIN0207_L6.3mm_D2.5mm_P7.62mm_Horizontal -> Resistor_SMD:R_0603_1608Metric
- R15, R23: value 1M -> 10k; footprint Resistor_THT:R_Axial_DIN0207_L6.3mm_D2.5mm_P7.62mm_Horizontal -> Resistor_SMD:R_0603_1608Metric
- R24: value 1M -> 330; footprint Resistor_THT:R_Axial_DIN0207_L6.3mm_D2.5mm_P7.62mm_Horizontal -> Resistor_SMD:R_0603_1608Metric
- SW11: footprint BDMLibrary:SW_Toggle_Blue_wSlots -> Button_Switch_THT:SW_PUSH_6mm
- U5: footprint Package_DIP:DIP-40_W15.24mm -> Package_DIP:DIP-40_W15.24mm_Socket
- moved J1 194.8 mm to (222.2, 15.0)
- moved SW11 176.0 mm to (227.4, 60.2)
- moved J2 163.8 mm to (205.6, 15.0)
- moved J14 149.0 mm to (72.3, 15.0)
- moved SW1 148.5 mm to (230.6, 80.3)
- moved R6 146.3 mm to (223.8, 42.5), turned to -90 degrees
- moved C1 142.9 mm to (61.5, 23.6), turned to -90 degrees
- moved R9 142.8 mm to (196.1, 51.6), turned to -90 degrees
- moved D5 140.2 mm to (55.1, 36.3)
- moved J3 132.9 mm to (188.9, 15.0)
- moved D6 131.5 mm to (45.0, 56.4)
- moved C4 130.2 mm to (67.9, 41.9), turned to 180 degrees
- moved R5 129.2 mm to (226.7, 42.4), turned to 90 degrees
- moved D4 128.0 mm to (103.0, 43.1)
- moved U2 127.4 mm to (61.5, 38.7), turned to -90 degrees
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Connections:
- C12 pad 1: GND -> VCC
- C12 pad 2: VCC -> GND
- C3 pad 1: Net-(C1-Pad1) -> GND
- C3 pad 2: GND -> /RST
- C7 pad 1: VCC -> Net-(C7-Pad1)
- D5 pad 1: GND -> Net-(D5-Pad1)
- D5 pad 2: /S33 -> VCC
- D6 pad 2: /S42 -> Net-(D6-Pad2)
- J10 pad 1: (no net) -> /MISO
- J10 pad 2: (no net) -> VCC
- J10 pad 3: (no net) -> /SCK
- R15 pad 1: /Vr -> VCC
- R15 pad 2: Net-(R15-Pad2) -> /RST
- R23 pad 1: /Vr -> Net-(D5-Pad1)
- R23 pad 2: Net-(J10-PadT) -> GND
- R24 pad 1: /Vr -> /SCK
- R24 pad 2: Net-(R24-Pad2) -> Net-(D6-Pad2)
- SW1 pad 1: GND -> VCC
- SW1 pad 2: Net-(SW1-Pad2) -> /FS1
- SW1 pad 3: VCC -> GND
- SW11 pad 2: VCC -> GND
- SW2 pad 1: GND -> VCC
- SW2 pad 2: Net-(SW2-Pad2) -> /FS2
- SW2 pad 3: VCC -> GND
- SW3 pad 1: GND -> VCC
- SW3 pad 2: Net-(SW3-Pad2) -> /FS3
- SW3 pad 3: VCC -> GND
- SW4 pad 1: GND -> VCC
- SW4 pad 2: Net-(SW4-Pad2) -> /FS4
- SW4 pad 3: VCC -> GND
- U2 pad 3: Net-(C1-Pad1) -> VCC
- U30 pad 15: Net-(R15-Pad2) -> Net-(C13-Pad1)
- U30 pad 3: Net-(R24-Pad2) -> unconnected-(U30-Pad3)
- U30 pad 4: Net-(R15-Pad2) -> unconnected-(U30-Pad4)
- U30 pad 5: Net-(J10-PadT) -> unconnected-(U30-Pad5)
- U5 pad 1: /S31 -> unconnected-(U5-Pad1)
- U5 pad 14: Net-(M1-Pad7) -> /LA
- U5 pad 15: Net-(M1-Pad6) -> /LB
- U5 pad 16: Net-(M1-Pad4) -> /LC
- U5 pad 17: Net-(M1-Pad2) -> /DA
- U5 pad 18: Net-(M1-Pad1) -> /DB
- U5 pad 19: Net-(M1-Pad9) -> /DC
- U5 pad 2: /S32 -> unconnected-(U5-Pad2)
- U5 pad 20: Net-(M1-Pad10) -> /DD
- U5 pad 21: Net-(M1-Pad5) -> /DDP
- U5 pad 22: Net-(SW12-Pad2) -> /FS1
- U5 pad 23: Net-(SW1-Pad2) -> /FS2
- U5 pad 24: Net-(SW2-Pad2) -> /FS3
- U5 pad 25: Net-(SW3-Pad2) -> /FS4
- U5 pad 26: Net-(SW4-Pad2) -> unconnected-(U5-Pad26)
- U5 pad 27: Net-(SW5-Pad2) -> unconnected-(U5-Pad27)
- U5 pad 28: Net-(SW6-Pad2) -> unconnected-(U5-Pad28)
- U5 pad 3: /S33 -> unconnected-(U5-Pad3)
- U5 pad 32: unconnected-(U5-Pad32) -> Net-(C7-Pad1)
- U5 pad 33: unconnected-(U5-Pad33) -> /S32
- U5 pad 34: unconnected-(U5-Pad34) -> /S31
- U5 pad 4: /S41 -> unconnected-(U5-Pad4)
- U5 pad 5: /S42 -> unconnected-(U5-Pad5)
- U5 pad 6: /S43 -> /MOSI
- U5 pad 7: unconnected-(U5-Pad7) -> /MISO
- U5 pad 8: unconnected-(U5-Pad8) -> /SCK
- U5 pad 9: VCC -> /RST
Routing:
- net /Vr: track 0.00 -> 76.2 mm
- net VCC: track 0.00 -> 73.0 mm
- net Net-(C13-Pad1): track 0.00 -> 38.2 mm, vias 0 -> 1
- net Net-(J8-PadT): track 0.00 -> 29.6 mm
- net Net-(C1-Pad1): track 0.00 -> 22.0 mm
- net Net-(J9-PadT): track 0.00 -> 19.5 mm
- net Net-(C13-Pad2): track 0.00 -> 12.0 mm
- net Net-(R20-Pad1): track 0.00 -> 10.8 mm
- net Net-(R3-Pad2): track 0.00 -> 8.84 mm
- net Net-(R1-Pad2): track 0.00 -> 5.86 mm
- net Net-(D5-Pad1): track 0.00 -> 2.68 mm
- net Net-(D6-Pad2): track 0.00 -> 2.45 mm
- added copper zone on F.Cu, net GND
Other:
- board outline added: 197.6 x 70.1 mm

Commit message: Update PCB
Parts:
- added R25: 470, Resistor_SMD:R_0603_1608Metric, F.Cu at (188.3, 115.7)
- added R27: 470, Resistor_SMD:R_0603_1608Metric, F.Cu at (158.3, 119.8)
- added R28: 470, Resistor_SMD:R_0603_1608Metric, F.Cu at (124.9, 119.8)
- added R29: 470, Resistor_SMD:R_0603_1608Metric, F.Cu at (88.4, 115.8)
- added R31: 470, Resistor_SMD:R_0603_1608Metric, F.Cu at (163.6, 131.7)
- added R40: 470, Resistor_SMD:R_0603_1608Metric, F.Cu at (103.1, 131.9)
- added R41: 470, Resistor_SMD:R_0603_1608Metric, F.Cu at (42.6, 131.8)
- C12: moved to F.Cu
- C5, C6: value 22pF -> 12pF
- J1, J14, J2, J3, J4, J5, J6, J7, J8, J9: footprint BDMLibrary:Mono Female Socket Connector TS -> BDMLibrary:Jack_6.35mm_Neutrik_NRJ4HF_Horizontal; moved to B.Cu
- R13, R17, R20, R7, R9: moved to B.Cu
- R23: value 10k -> 470
- R24: value 330 -> 470
- Y1: value 12MHz -> 16MHz; footprint Crystal:Crystal_HC49-U_Vertical -> Crystal:Crystal_SMD_3225-4Pin_3.2x2.5mm
- moved C6 105.7 mm to (74.2, 142.1), turned to 90 degrees
- moved Y1 102.2 mm to (78.0, 142.1), turned to 180 degrees
- moved C5 97.8 mm to (81.9, 142.1), turned to -90 degrees
- moved C12 94.7 mm to (73.4, 139.4)
- moved C11 92.4 mm to (158.4, 134.6)
- moved R14 92.4 mm to (165.7, 122.9)
- moved U5 92.0 mm to (48.8, 137.1)
- moved R9 91.9 mm to (178.9, 141.8), turned to 90 degrees
- moved R7 91.4 mm to (184.7, 142.4), turned to 90 degrees
- moved C10 91.0 mm to (133.9, 134.6), turned to -90 degrees
- moved R20 90.8 mm to (159.2, 124.0)
- moved J1 90.1 mm to (231.1, 104.6), turned to 90 degrees
- moved J2 90.0 mm to (213.4, 104.6), turned to 90 degrees
- moved J3 89.9 mm to (195.6, 104.6), turned to 90 degrees
- moved J4 89.8 mm to (177.8, 104.6), turned to 90 degrees
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Connections:
- D1 pad 1: GND -> Net-(D1-Pad1)
- D10 pad 1: GND -> Net-(D10-Pad1)
- D11 pad 1: GND -> Net-(D11-Pad1)
- D2 pad 1: GND -> Net-(D2-Pad1)
- D3 pad 1: GND -> Net-(D3-Pad1)
- D4 pad 1: GND -> Net-(D4-Pad1)
- D9 pad 1: GND -> Net-(D9-Pad1)
- Y1 pad 2: Net-(C6-Pad1) -> GND
Routing:
- net /Vr: track 76.2 -> 183.8 mm
- net /RST: track 0.00 -> 45.0 mm
- net /SCK: track 0.00 -> 38.5 mm
- net Net-(C13-Pad1): track 38.2 -> 4.12 mm, vias 1 -> 0
- net /MISO: track 0.00 -> 30.0 mm
- net Net-(J8-PadT): track 29.6 -> 2.98 mm
- net /MOSI: track 0.00 -> 23.9 mm
- net Net-(J9-PadT): track 19.5 -> 2.96 mm
- net Net-(C8-Pad1): track 0.00 -> 13.6 mm
- net Net-(R20-Pad1): track 10.8 -> 0.00 mm
- net Net-(C6-Pad1): track 0.00 -> 9.60 mm
- net Net-(C5-Pad1): track 0.00 -> 7.03 mm
- net Net-(C8-Pad2): track 0.00 -> 5.50 mm
- net Net-(D11-Pad1): track 0.00 -> 4.04 mm
- net Net-(C13-Pad2): track 12.0 -> 15.3 mm
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Other:
- board size 197.6 x 70.1 mm -> 201.4 x 60.1 mm
