File: kicad/PedalComposer.kicad_sch (KiCad schematic)
At the start: 82 parts, among them J1 In, J10 Fx5In, J11 Fx5Out, J12 Fx6In, J13 Fx6Out, J14 Out, J15 Jack-DC, J2 Fx1In, J3 Fx1Out, J4 Fx2In, J5 Fx2Out, J6 Fx3In, J7 Fx3Out, J8 Fx4In, J9 Fx4Out, M1 7-SEGMENT-1DIGIT-1INCH-BLUE, SW1 Fx1, SW11 Edit, SW12 All, SW2 Fx2, SW3 Fx3, SW4 Fx4, SW5 Fx5, SW6 Fx6, U1 LM317L_TO92, U10 CD4053B, U20 CD4053B, U30 CD4053B, U40 CD4053B, U5 ATmega8535-16P, Y1 8MHz

Commit message: Update sch, down to 4 Fx
Parts:
- removed C1, C3: 100pF, Capacitor_THT:C_Radial_D6.3mm_H11.0mm_P2.50mm, symbol darkglass-microtubes-b3k-rescue:CP-Device
- removed C? (x2): 1uF, symbol Device:C
- removed D? (x2): LED, symbol Device:LED
- removed J10: Fx5In, symbol Connector:AudioJack2
- removed J11: Fx5Out, symbol Connector:AudioJack2
- removed J12: Fx6In, symbol Connector:AudioJack2
- removed J13: Fx6Out, symbol Connector:AudioJack2
- removed R? (x8): 1M, symbol Device:R
- removed SW12: All, symbol Switch:SW_SPDT
- removed SW5: Fx5, symbol Switch:SW_Push_SPDT
- removed SW6: Fx6, symbol Switch:SW_Push_SPDT
- removed U40: CD4053B, symbol Analog_Switch:CD4053B
- added C1, C12, C7: 100nF, symbol Device:C
- added C3: 10nF, Capacitor_THT:C_Rect_L7.2mm_W3.0mm_P5.00mm_FKS2_FKP2_MKS2_MKP2, symbol Device:C
- added D10, D11, D5, D9: LED, symbol Device:LED
- added D6: LED, LED_THT:LED_D3.0mm, symbol Device:LED
- added J10: AVR-ISP-6, Connector_PinHeader_2.54mm:PinHeader_2x03_P2.54mm_Vertical, symbol Connector:AVR-ISP-6
- added R15, R23: 10k, symbol Device:R
- added R24: 330, symbol Device:R
- added R32, R33, R34, R35, R36, R37, R38, R39: 470, symbol Device:R
- added U3: 4543, symbol 4xxx:4543
- C10, C11, C9: renamed from C?; value 1uF -> 100nF; footprint (none) -> Capacitor_THT:C_Rect_L7.2mm_W3.0mm_P5.00mm_FKS2_FKP2_MKS2_MKP2
- C13: renamed from C?; footprint (none) -> Capacitor_THT:C_Rect_L7.2mm_W3.0mm_P5.00mm_FKS2_FKP2_MKS2_MKP2
- C5, C6: renamed from C?; footprint (none) -> Capacitor_THT:C_Disc_D5.0mm_W2.5mm_P5.00mm
- C8: renamed from C?; value 2.2uF -> 100nF; footprint (none) -> Capacitor_THT:C_Rect_L7.2mm_W3.0mm_P5.00mm_FKS2_FKP2_MKS2_MKP2
- D1, D2, D3, D4: renamed from D?; footprint (none) -> LED_THT:LED_D3.0mm
- J1, J14: footprint (none) -> BDMLibrary:Mono Female Socket Connector
- J2: value Fx1In -> Send1; footprint (none) -> BDMLibrary:Mono Female Socket Connector
- J3: value Fx1Out -> Return1; footprint (none) -> BDMLibrary:Mono Female Socket Connector
- J4: value Fx2In -> Send2; footprint (none) -> BDMLibrary:Mono Female Socket Connector
- J5: value Fx2Out -> Return2; footprint (none) -> BDMLibrary:Mono Female Socket Connector
- J6: value Fx3In -> Send3; footprint (none) -> BDMLibrary:Mono Female Socket Connector
- J7: value Fx3Out -> Return3; footprint (none) -> BDMLibrary:Mono Female Socket Connector
- J8: value Fx4In -> Send4; footprint (none) -> BDMLibrary:Mono Female Socket Connector
- J9: value Fx4Out -> Return4; footprint (none) -> BDMLibrary:Mono Female Socket Connector
- M1: footprint 7-SEGMENT-1DIGIT-PTH -> Display_7Segment:7SegmentLED_LTS6760_LTS6780
- R10, R11, R12, R13, R14, R16, R17, R18, R19, R20, R21, R22, R26, R30, R5, R6, R7, R8, R9: renamed from R?; footprint (none) -> Resistor_THT:R_Axial_DIN0207_L6.3mm_D2.5mm_P7.62mm_Horizontal
- SW1, SW2, SW3, SW4: footprint (none) -> BDMLibrary:SW_Toggle_Blue_wSlots
- SW11: footprint (none) -> Button_Switch_THT:SW_PUSH_6mm
- U10, U20, U30: footprint (none) -> Package_DIP:DIP-16_W7.62mm_Socket
- Y1: value 8MHz -> 12MHz; footprint (none) -> Crystal:Crystal_HC49-U_Vertical
- gave numbers to parts that had none: 1
Connections:
- net GND: now also C10.1, C11.1, C9.1, M1.3 (G1), M1.8 (G2), SW1.3 (C), SW11.2, SW2.3 (C), SW3.3 (C), SW4.3 (C), C1.2, C12.2, C3.1, C7.2, D10.1 (K), D11.1 (K), D6.1 (K), D9.1 (K), J10.6 (GND), R23.2, U3.1 (~{LE}), U3.8 (VSS); no longer SW1.1 (A), SW2.1 (A), SW3.1 (A), SW4.1 (A)
- net S31: now also U5.34 (PA6); no longer U5.1 (PB0)
- net S32: now also U5.33 (PA7); no longer U5.2 (PB1)
- net S33: no longer U5.3 (PB2)
- net VCC: now also C10.2, C11.2, C9.2, SW1.1 (A), SW2.1 (A), SW3.1 (A), SW4.1 (A), U10.16 (VDD), U2.3 (VI), U20.16 (VDD), U30.16 (VDD), U5.10 (VCC), U5.30 (AVCC), C12.1, D5.2 (A), J10.2 (VCC), R15.1, U3.16 (VDD), U3.6 (PH), U3.7 (BL); no longer C10.1, C11.1, C9.1, M1.3 (G1), M1.8 (G2), SW1.3 (C), SW11.2, SW2.3 (C), SW3.3 (C), SW4.3 (C)
- net at J15.2, U1.3 (VI): now also C1.1; no longer U2.3 (VI)
- net at M1.1 (E): now also R36.2; no longer U5.18 (PD4)
- net at M1.10 (G): now also R38.2; no longer U5.20 (PD6)
- net at M1.2 (D): now also R35.2; no longer U5.17 (PD3)
- net at M1.4 (C): now also R34.2; no longer U5.16 (PD2)
- net at M1.5 (DP): now also R39.2; no longer U5.21 (PD7)
- net at M1.6 (B): now also R33.2; no longer U5.15 (PD1)
- net at M1.7 (A): now also R32.2; no longer U5.14 (PD0)
- net at M1.9 (F): now also R37.2; no longer U5.19 (PD5)
- net at U30.15 (B): now also C13.1, R26.2; no longer U30.4 (C)
- net FS1: now reaches U5.22 (PC0)
- net FS1: now also SW1.2 (B)
- net FS2: now reaches U5.23 (PC1)
- net FS2: now also SW2.2 (B); no longer SW1.2 (B)
- net FS3: now reaches U5.24 (PC2)
- net FS3: now also SW3.2 (B); no longer SW2.2 (B)
- net FS4: now reaches U5.25 (PC3)
- net FS4: now also SW4.2 (B); no longer SW3.2 (B)
- net at U5.26 (PC4): no longer SW4.2 (B)
- net at U5.32 (AREF): now also C7.1
- net MISO: now reaches U5.7 (PB6)
- net MISO: now also J10.1 (MISO)
- net SCK: now reaches U5.8 (PB7)
- net SCK: now also J10.3 (SCK), R24.1
- net S41: no longer names the net of U5.4 (PB3)
- net S42: no longer names the net of U5.5 (PB4)
- net S43 renamed MOSI
- net MOSI: now also J10.4 (MOSI)
- new net: D6.2 (A), R24.2
- new net: R37.1, U3.15 (Qf)
- new net: C3.2, J10.5 (~{RST}), R15.2, U5.9 (~{RESET})
- new net: D5.1 (K), R23.1
- new net: R33.1, U3.10 (Qb)
- new net: R34.1, U3.11 (Qc)
- new net: R35.1, U3.12 (Qd)
- new net: R36.1, U3.13 (Qe)
- new net: R38.1, U3.14 (Qg)
- new net: R32.1, U3.9 (Qa)
- new net DA: U3.5 (D0), U5.17 (PD3)
- new net DB: U3.3 (D1), U5.18 (PD4)
- new net DC: U3.2 (D2), U5.19 (PD5)
- new net DD: U3.4 (D3), U5.20 (PD6)
- new net DDP: R39.1, U5.21 (PD7)
- new net LA: D9.2 (A), U5.14 (PD0)
- new net LB: D10.2 (A), U5.15 (PD1)
- new net LC: D11.2 (A), U5.16 (PD2)
- no-connect marks 0 -> 8
Other:
- moved on the sheet: C10, C11, C13, C2, C4, C5, C6, C8, C9, D1, D2, D3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

Commit message: WIP layout
Parts:
- C1, C12, C7: footprint (none) -> Capacitor_SMD:C_0603_1608Metric
- C10, C11, C3, C9: footprint Capacitor_THT:C_Rect_L7.2mm_W3.0mm_P5.00mm_FKS2_FKP2_MKS2_MKP2 -> Capacitor_SMD:C_0603_1608Metric
- C13: footprint Capacitor_THT:C_Rect_L7.2mm_W3.0mm_P5.00mm_FKS2_FKP2_MKS2_MKP2 -> Capacitor_SMD:C_Elec_4x5.4
- C2, C4: footprint Capacitor_THT:C_Radial_D6.3mm_H11.0mm_P2.50mm -> Capacitor_SMD:C_Elec_4x5.4
- C5, C6: footprint Capacitor_THT:C_Disc_D5.0mm_W2.5mm_P5.00mm -> Capacitor_SMD:C_0603_1608Metric
- C8: value 100nF -> 2.2uF; footprint Capacitor_THT:C_Rect_L7.2mm_W3.0mm_P5.00mm_FKS2_FKP2_MKS2_MKP2 -> Capacitor_SMD:C_Elec_4x5.4
- D1: value LED -> Fx1
- D10: value LED -> Ctrl2; footprint (none) -> LED_THT:LED_D3.0mm
- D11: value LED -> Ctrl3; footprint (none) -> LED_THT:LED_D3.0mm
- D2: value LED -> Fx2
- D3: value LED -> Fx3
- D4: value LED -> Fx4
- D5: footprint (none) -> LED_SMD:LED_0603_1608Metric
- D6: footprint LED_THT:LED_D3.0mm -> LED_SMD:LED_0603_1608Metric
- D9: value LED -> Ctrl1; footprint (none) -> LED_THT:LED_D3.0mm
- J1, J14, J2, J3, J4, J5, J6, J7, J8, J9: footprint BDMLibrary:Mono Female Socket Connector -> BDMLibrary:Mono Female Socket Connector TS
- R1, R10, R11, R12, R13, R14, R16, R17, R18, R19, R2, R20, R21, R22, R26, R3, R30, R4, R5, R6, R7, R8, R9: footprint Resistor_THT:R_Axial_DIN0207_L6.3mm_D2.5mm_P7.62mm_Horizontal -> Resistor_SMD:R_0603_1608Metric
- R15, R23, R24, R32, R33, R34, R35, R36, R37, R38, R39: footprint (none) -> Resistor_SMD:R_0603_1608Metric
- U3: footprint (none) -> Package_SO:SOIC-16_4.55x10.3mm_P1.27mm
- U5: footprint Package_DIP:DIP-40_W15.24mm -> Package_DIP:DIP-40_W15.24mm_Socket
Connections:
- net RST: now reaches C3.2, J10.5 (~{RST}), R15.2, U5.9 (~{RESET})
Other:
- moved on the sheet: C1, C12, C2, C3, C4, C5, C6, C7, D1, D10, D11, D2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

Commit message: Update PCB
Parts:
- removed Y1: 12MHz, Crystal:Crystal_HC49-U_Vertical, symbol Device:Crystal
- added R25, R27, R28, R29, R31, R40, R41: 470, Resistor_SMD:R_0603_1608Metric, symbol Device:R
- added Y1: 16MHz, Crystal:Crystal_SMD_3225-4Pin_3.2x2.5mm, symbol Device:Crystal_GND24
- C5, C6: value 22pF -> 12pF
- J1, J14, J2, J3, J4, J5, J6, J7, J8, J9: footprint BDMLibrary:Mono Female Socket Connector TS -> BDMLibrary:Jack_6.35mm_Neutrik_NRJ4HF_Horizontal
- R23: value 10k -> 470
- R24: value 330 -> 470
Connections:
- net GND: now also R25.1, R27.1, R28.1, R29.1, R31.1, R40.1, R41.1, Y1.2, Y1.4; no longer D1.1 (K), D10.1 (K), D11.1 (K), D2.1 (K), D3.1 (K), D4.1 (K), D9.1 (K)
- net at C5.1, U5.13 (XTAL1): now also Y1.1
- net at C6.1, U5.12 (XTAL2): now also Y1.3
- new net: D2.1 (K), R27.2
- new net: D11.1 (K), R41.2
- new net: D10.1 (K), R40.2
- new net: D4.1 (K), R29.2
- new net: D1.1 (K), R25.2
- new net: D9.1 (K), R31.2
- new net: D3.1 (K), R28.2
