File: kicad/ctrl_board/ctrl_board.kicad_pcb (KiCad board)
At the start: 2 copper layers, 198.1 x 18.4 mm, 11 parts, among them J1 Conn_Ctrl, SW1 SW1, SW2 SW2, SW3 SW3, SW4 SW4

Commit message: Boards v1
Parts:
- R2, R3, R4: footprint Resistor_SMD:R_0603_1608Metric -> Resistor_THT:R_Axial_DIN0207_L6.3mm_D2.5mm_P7.62mm_Horizontal
- moved R4 8.26 mm to (65.2, 93.1), turned to 0 degrees
- moved D4 2.42 mm to (62.1, 93.2), turned to 180 degrees
Routing:
- net /LC: track 88.4 -> 91.0 mm
- net Net-(D4-Pad1): track 1.96 -> 3.10 mm
