File: kicad/ctrl_board/ctrl_board.kicad_sch (KiCad schematic)
At the start: 11 parts, among them J1 Conn_Ctrl, SW1 SW1, SW2 SW2, SW3 SW3, SW4 SW4

Commit message: Boards v1
Parts:
- R2, R3, R4: footprint Resistor_SMD:R_0603_1608Metric -> Resistor_THT:R_Axial_DIN0207_L6.3mm_D2.5mm_P7.62mm_Horizontal
Changed lines of the file:
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@@
     (property "Reference" "R4" (id 0) (at 111.76 97.79 90))
     (property "Value" "470" (id 1) (at 111.76 100.33 90))
-    (property "Footprint" "Resistor_SMD:R_0603_1608Metric" (id 2) (at 111.76 105.918 90)
+    (property "Footprint" "Resistor_THT:R_Axial_DIN0207_L6.3mm_D2.5mm_P7.62mm_Horizontal" (id 2) (at 111.76 105.918 90)
       (effects (font (size 1.27 1.27)) hide)
     )
@@
     (property "Reference" "R3" (id 0) (at 111.76 87.63 90))
     (property "Value" "470" (id 1) (at 111.76 90.17 90))
-    (property "Footprint" "Resistor_SMD:R_0603_1608Metric" (id 2) (at 111.76 95.758 90)
+    (property "Footprint" "Resistor_THT:R_Axial_DIN0207_L6.3mm_D2.5mm_P7.62mm_Horizontal" (id 2) (at 111.76 95.758 90)
       (effects (font (size 1.27 1.27)) hide)
     )
@@
   (symbol (lib_id "power:GND") (at 36.83 72.39 0) (unit 1)
     (in_bom yes) (on_board yes) (fields_autoplaced)
-    (property "Reference" "#PWR?" (id 0) (at 36.83 78.74 0)
+    (property "Reference" "#PWR0103" (id 0) (at 36.83 78.74 0)
       (effects (font (size 1.27 1.27)) hide)
     )
@@
   (symbol (lib_id "power:VCC") (at 36.83 46.99 0) (unit 1)
     (in_bom yes) (on_board yes) (fields_autoplaced)
-    (property "Reference" "#PWR?" (id 0) (at 36.83 50.8 0)
+    (property "Reference" "#PWR0102" (id 0) (at 36.83 50.8 0)
       (effects (font (size 1.27 1.27)) hide)
     )
@@
     (property "Reference" "R2" (id 0) (at 111.76 77.47 90))
     (property "Value" "470" (id 1) (at 111.76 80.01 90))
-    (property "Footprint" "Resistor_SMD:R_0603_1608Metric" (id 2) (at 111.76 85.598 90)
+    (property "Footprint" "Resistor_THT:R_Axial_DIN0207_L6.3mm_D2.5mm_P7.62mm_Horizontal" (id 2) (at 111.76 85.598 90)
       (effects (font (size 1.27 1.27)) hide)
     )
@@
   (symbol (lib_id "power:GND") (at 116.84 106.68 0) (unit 1)
     (in_bom yes) (on_board yes) (fields_autoplaced)
-    (property "Reference" "#PWR?" (id 0) (at 116.84 113.03 0)
+    (property "Reference" "#PWR0101" (id 0) (at 116.84 113.03 0)
       (effects (font (size 1.27 1.27)) hide)
     )
@@
       (reference "#PWR01") (unit 1) (value "VCC") (footprint "")
     )
+    (path "/facb8cff-e8e4-40a5-afc4-c266ee63af67"
+      (reference "#PWR0101") (unit 1) (value "GND") (footprint "")
+    )
+    (path "/d129d375-8b04-439f-a139-6bf5f17a61f1"
+      (reference "#PWR0102") (unit 1) (value "VCC") (footprint "")
+    )
     (path "/88d04aa0-a5f1-43df-9656-fb4c3b50e96e"
-      (reference "#PWR?") (unit 1) (value "GND") (footprint "")
-    )
-    (path "/d129d375-8b04-439f-a139-6bf5f17a61f1"
-      (reference "#PWR?") (unit 1) (value "VCC") (footprint "")
-    )
-    (path "/facb8cff-e8e4-40a5-afc4-c266ee63af67"
-      (reference "#PWR?") (unit 1) (value "GND") (footprint "")
+      (reference "#PWR0103") (unit 1) (value "GND") (footprint "")
     )
     (path "/bf4311fa-861b-4f3e-b3fb-8fd1e4798c48"
@@
     )
     (path "/daa676a9-1e0f-4dca-88a2-e0227a6671aa"
-      (reference "R2") (unit 1) (value "470") (footprint "Resistor_SMD:R_0603_1608Metric")
+      (reference "R2") (unit 1) (value "470") (footprint "Resistor_THT:R_Axial_DIN0207_L6.3mm_D2.5mm_P7.62mm_Horizontal")
     )
     (path "/3abc7555-7cbd-403a-bdee-12a76f17b279"
-      (reference "R3") (unit 1) (value "470") (footprint "Resistor_SMD:R_0603_1608Metric")
+      (reference "R3") (unit 1) (value "470") (footprint "Resistor_THT:R_Axial_DIN0207_L6.3mm_D2.5mm_P7.62mm_Horizontal")
     )
     (path "/09c6c498-5837-4f03-b640-93be131ca3ba"
-      (reference "R4") (unit 1) (value "470") (footprint "Resistor_SMD:R_0603_1608Metric")
+      (reference "R4") (unit 1) (value "470") (footprint "Resistor_THT:R_Axial_DIN0207_L6.3mm_D2.5mm_P7.62mm_Horizontal")
     )
     (path "/0bb927d2-4731-4b52-84c0-dd32b78965f9"
