File: kicad/main_board/PedalComposer.kicad_pcb (KiCad board)
At the start: 2 copper layers, 201 x 55.5 mm, 81 parts, among them J1 In, J10 AVR-ISP-6, J11 Conn_Ctrl, J14 Out, J15 Jack-DC, J2 Send1, J3 Return1, J4 Send2, J5 Return2, J6 Send3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

Commit message: Boards v1
Parts:
- added D7: SM4001, Diode_SMD:D_SOD-123F, F.Cu at (30.0, 41.7)
- added D8: SM4001, Diode_SMD:D_SOD-123F, F.Cu at (37.1, 57.0)
- C13, C8: footprint Capacitor_SMD:C_Elec_4x5.4 -> Capacitor_SMD:C_0805_2012Metric
- C2, C4: footprint Capacitor_SMD:C_Elec_4x5.4 -> Capacitor_SMD:CP_Elec_4x5.4
- U3: value 4543 -> CD4543BM96
- moved R26 2.08 mm to (60.0, 54.7)
- moved C13 1.80 mm to (57.0, 53.8)
- moved C8 0.71 mm to (214.2, 54.5)
- moved C4 0.26 mm to (42.8, 53.9)
Routing:
- net VCC: track 281.4 -> 289.8 mm
- net Net-(C1-Pad1): track 20.9 -> 28.1 mm
- net /Vr: track 234.6 -> 239.4 mm
- net Net-(C13-Pad2): track 15.3 -> 14.2 mm
- net Net-(C8-Pad1): track 13.6 -> 14.2 mm
- net Net-(C13-Pad1): track 49.9 -> 49.4 mm
