File: kicad/main_board/PedalComposer.kicad_sch (KiCad schematic)
At the start: 89 parts, among them J1 In, J10 AVR-ISP-6, J14 Out, J15 Jack-DC, J2 Send1, J3 Return1, J4 Send2, J5 Return2, J6 Send3, J7 Return3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

Commit message: Update PCB
Parts:
- removed D10: Ctrl2, LED_THT:LED_D3.0mm, symbol Device:LED
- removed D11: Ctrl3, LED_THT:LED_D3.0mm, symbol Device:LED
- removed D9: Ctrl1, LED_THT:LED_D3.0mm, symbol Device:LED
- removed R40, R41: 470, Resistor_SMD:R_0603_1608Metric, symbol Device:R
- removed SW1: Fx1, BDMLibrary:SW_Toggle_Blue_wSlots, symbol Switch:SW_Push_SPDT
- removed SW2: Fx2, BDMLibrary:SW_Toggle_Blue_wSlots, symbol Switch:SW_Push_SPDT
- removed SW3: Fx3, BDMLibrary:SW_Toggle_Blue_wSlots, symbol Switch:SW_Push_SPDT
- removed SW4: Fx4, BDMLibrary:SW_Toggle_Blue_wSlots, symbol Switch:SW_Push_SPDT
- added J11: Conn_Ctrl, Connector_PinHeader_2.54mm:PinHeader_1x10_P2.54mm_Vertical, symbol Connector:Conn_01x10_Female
- R31: value 470 -> 10k
- U3: footprint Package_SO:SOIC-16_4.55x10.3mm_P1.27mm -> Package_SO:SOIC-16_3.9x9.9mm_P1.27mm
Connections:
- net FS1 is gone; now on net S32: U5.22 (PC0)
- net FS2 is gone; now on net S23: U5.23 (PC1)
- net FS3 is gone; now on net S22: U5.24 (PC2)
- net FS4 is gone; now on net S21: U5.25 (PC3)
- net DA: now also U5.20 (PD6); no longer U5.17 (PD3)
- net DC: now also U5.17 (PD3); no longer U5.19 (PD5)
- net DD: now also U5.19 (PD5); no longer U5.20 (PD6)
- net DDP: now also U5.16 (PD2); no longer U5.21 (PD7)
- net GND: now also R31.2, U30.11 (S1), U30.12 (A0), U30.13 (A1), U30.14 (A), J11.10 (Pin_10); no longer R31.1, SW11.2
- net LA: now also U5.39 (PA1), J11.3 (Pin_3); no longer U5.14 (PD0)
- net LB: now also U5.38 (PA2), J11.5 (Pin_5); no longer U5.15 (PD1)
- net LC: now also U5.37 (PA3), J11.7 (Pin_7); no longer U5.16 (PD2)
- net S11: now also U5.28 (PC6); no longer U5.40 (PA0)
- net S12: now also U5.27 (PC5); no longer U5.39 (PA1)
- net S13: now also U5.26 (PC4); no longer U5.38 (PA2)
- net S21: no longer U5.37 (PA3)
- net S22: no longer U5.36 (PA4)
- net S23: no longer U5.35 (PA5)
- net S32: now also D4.2 (A); no longer U5.33 (PA7)
- net S33: now also U5.21 (PD7)
- net VCC: now also SW11.2, J11.1 (Pin_1)
- net at J9.T, R21.2: now also U30.5 (C0); no longer U30.2 (B0)
- net at R14.2, U20.4 (C): now also U30.15 (B); no longer U30.14 (A)
- net at J8.T, R18.2: now also U30.2 (B0); no longer U30.12 (A0)
- net at R20.1, U30.1 (B1): now also U30.3 (C1); no longer U30.13 (A1)
- net at C13.1, R26.2: now also U30.4 (C); no longer U30.15 (B)
- net FSw1: now reaches U5.1 (PB0)
- net FSw1: now also J11.2 (Pin_2)
- net FSw2: now reaches U5.2 (PB1)
- net FSw2: now also J11.4 (Pin_4)
- net SWEdit: now reaches SW11.1, U5.29 (PC7)
- net SWEdit: now also R31.1
- net FSw3: now reaches U5.3 (PB2)
- net FSw3: now also J11.6 (Pin_6)
- net FSw4: now reaches U5.5 (PB4)
- net FSw4: now also J11.8 (Pin_8)
- removed net S31: D4.2 (A), U30.11 (S1), U5.34 (PA6)
- no-connect marks 8 -> 9
Other:
- moved on the sheet: SW11

Commit message: Boards v1
Parts:
- added D7, D8: SM4002, Diode_SMD:D_SOD-123F, symbol Diode:SM4001
- C1, C10, C11, C12, C7, C9: LCSC (none) -> C14663; Manufacturer (none) -> JLC
- C13, C8: footprint Capacitor_SMD:C_Elec_4x5.4 -> Capacitor_SMD:C_0805_2012Metric; LCSC (none) -> C19110; Manufacturer (none) -> JLC
- C2, C4: footprint Capacitor_SMD:C_Elec_4x5.4 -> Capacitor_SMD:CP_Elec_4x5.4; LCSC (none) -> C72491
- C3: LCSC (none) -> C100042; Manufacturer (none) -> JLC
- C5, C6: LCSC (none) -> C38523; Manufacturer (none) -> JLC
- D5, D6: LCSC (none) -> C2297; Manufacturer (none) -> JLC
- J10: LCSC (none) -> C65114
- J11: LCSC (none) -> C57369
- J15: Manufacturer JLC -> (none)
- R1: LCSC (none) -> C23138
- R10, R11, R12, R13, R14, R16, R17, R18, R19, R20, R21, R22, R26, R30, R5, R6, R7, R8, R9: LCSC (none) -> C22935; Manufacturer (none) -> JLC
- R15, R31: LCSC (none) -> C25804; Manufacturer (none) -> JLC
- R2: LCSC (none) -> C21190
- R23, R24, R25, R27, R28, R29, R32, R33, R34, R35, R36, R37, R38, R39: LCSC (none) -> C23179; Manufacturer (none) -> JLC
- R3, R4: LCSC (none) -> C23179
- SW11: LCSC (none) -> C13828; Manufacturer (none) -> JLC
- U10, U20, U30: LCSC (none) -> C2326; Manufacturer (none) -> JLC
- U3: value 4543 -> CD4543BM96; LCSC (none) -> C28326; Manufacturer (none) -> JLC
- U5: LCSC (none) -> C2332; Manufacturer (none) -> JLC
- Y1: LCSC (none) -> C13738; Manufacturer (none) -> JLC
Connections:
- net VCC: now also D7.2 (A), D8.1 (K)
- net Vr: now also D8.2 (A)
- net at C1.1, J15.2, U1.3 (VI): now also D7.1 (K)
